File: PVDX-ADCS-Board.kicad_pcb (KiCad board)
At the start: 4 copper layers, 82.5 x 82.5 mm, 96 parts, among them J1 Conn_02x18_Row_Letter_Last, J2 Conn_01x18, J3 Conn_01x06, J4 Conn_01x02, J5 Conn_01x17, J6 Conn_01x03, J7 Conn_01x09, U1 TLV9001IDCK, U10 DRV8837C, U11 OPA2381AIDGKR, U12 OPA2381AIDGKR, U13 OPA2381AIDGKR, U14 OPA2381AIDGKR, U15 OPA2381AIDGKR, U16 OPA2381AIDGKR, U17 OPA2381AIDGKR, U18 OPA2381AIDGKR, U19 OPA2381AIDGKR, U2 INA226, U3 DRV8837C, U4 DRV8837C, U5 MCP23017x-x-SO, U6 ADG734BRUZ, U7 ADG734BRUZ, U8 ADG734BRUZ, U9 ADG734BRUZ

Commit message: 100% mtq, 85% pd, 90% pmb
Parts:
- added C1: 100n, Capacitor_SMD:C_0402_1005Metric, F.Cu at (217.2, 105.5)
- added C2: 100n, Capacitor_SMD:C_0402_1005Metric, F.Cu at (211.5, 105.5)
- added C3: 100n, Capacitor_SMD:C_0402_1005Metric, F.Cu at (205.7, 105.5)
- added C4: 100n, Capacitor_SMD:C_0402_1005Metric, F.Cu at (199.9, 105.5)
- added C5: 100n, Capacitor_SMD:C_0402_1005Metric, F.Cu at (194.1, 105.5)
- added C6: 100n, Capacitor_SMD:C_0402_1005Metric, F.Cu at (188.3, 105.5)
- added C7: 100n, Capacitor_SMD:C_0402_1005Metric, F.Cu at (182.5, 105.5)
- added C8: 100n, Capacitor_SMD:C_0402_1005Metric, F.Cu at (176.7, 105.5)
- added C9: 100n, Capacitor_SMD:C_0402_1005Metric, F.Cu at (170.9, 105.5)
- added CBY5: 100n, Capacitor_SMD:C_0402_1005Metric, F.Cu at (174.5, 73.5)
- added H1: MountingHole, footprints:MountingHole_3.4mm_M3_PVDX, F.Cu at (144.8, 42.2)
- added H2: MountingHole, footprints:MountingHole_3.4mm_M3_PVDX, F.Cu at (217.8, 42.2)
- added H3: MountingHole, footprints:MountingHole_3.4mm_M3_PVDX, F.Cu at (217.8, 115.2)
- added H4: MountingHole, footprints:MountingHole_3.4mm_M3_PVDX, F.Cu at (144.8, 115.2)
- C37, C38, C39, C40, C41, C42: value 0.1u -> 100n
- CBY2: renamed from C_BY2; value 0.1u -> 100n
- CBY6: renamed from C_BY6; value 0.1u -> 100n
- CBY7: renamed from C_BY7; value 0.1u -> 100n
- CBY8: renamed from C_BY8; value 0.1u -> 100n
- CBY9: renamed from C_BY9; value 0.1u -> 100n
- R10, R11, R12, R13, R14, R15, R16, R17, R18, R3, R4, R5, R6, R7, R8, R9: value 100 -> 100R
- R40, R41, R42, R43, R44, R45, R46, R47, R48, R49, R50, R51, R52, R53, R54, R55, R56, R57: value 2.2k -> 2k2
- RSH1: renamed from R_SHUNT1; value 10 -> 10R
- moved R57 93.1 mm to (167.6, 108.2), turned to 0 degrees
- moved C62 87.2 mm to (167.6, 109.8), turned to 0 degrees
- moved R56 86.7 mm to (169.9, 99.5), turned to 0 degrees
- moved R55 82.5 mm to (173.4, 108.2), turned to 0 degrees
- moved C61 82.0 mm to (169.9, 98.0), turned to 0 degrees
- moved C60 76.5 mm to (173.4, 109.8), turned to 0 degrees
- moved R54 76.0 mm to (175.7, 99.5), turned to 0 degrees
- moved R53 72.1 mm to (179.2, 108.2), turned to 0 degrees
- moved C59 71.2 mm to (175.7, 98.0), turned to 0 degrees
- moved C58 65.8 mm to (179.2, 109.8), turned to 0 degrees
- moved R48 65.8 mm to (193.1, 99.5), turned to 0 degrees
- moved R52 65.4 mm to (181.5, 99.5), turned to 0 degrees
- moved R51 61.8 mm to (185.0, 108.2), turned to 0 degrees
- moved C53 61.7 mm to (193.1, 98.0), turned to 0 degrees
- moved R47 61.6 mm to (196.5, 108.2), turned to 0 degrees
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Connections:
- J7 pad 1: MCTRL1_1 -> MSLEEP1
- J7 pad 2: MCTRL1_2 -> MCTRL1_1
- J7 pad 3: MSLEEP1 -> MCTRL1_2
- J7 pad 4: MCTRL2_1 -> MSLEEP2
- J7 pad 5: MCTRL2_2 -> MCTRL2_1
- J7 pad 6: MSLEEP2 -> MCTRL2_2
- J7 pad 7: MCTRL3_1 -> MSLEEP3
- J7 pad 8: MCTRL3_2 -> MCTRL3_1
- J7 pad 9: MSLEEP3 -> MCTRL3_2
- U5 pad 11: unconnected-(U5-NC-Pad11) -> GND
- U5 pad 14: unconnected-(U5-NC-Pad14) -> GND
Routing:
- net MCTRL3_2: track 0.00 -> 56.0 mm
- net MCTRL3_1: track 0.00 -> 53.9 mm
- net MSLEEP3: track 0.00 -> 51.7 mm
- net MCTRL2_2: track 0.00 -> 42.3 mm
- net MCTRL2_1: track 0.00 -> 40.1 mm
- net MSLEEP2: track 0.00 -> 37.9 mm
- net MCTRL1_2: track 0.00 -> 29.0 mm
- net MCTRL1_1: track 0.00 -> 26.8 mm
- net +3V3: track 54.8 -> 80.5 mm, vias 11 -> 21
- net GND: track 77.7 -> 103.1 mm, vias 25 -> 36
- net MSLEEP1: track 0.00 -> 24.6 mm
- net PD6: track 0.00 -> 4.34 mm
- net PD2: track 8.68 -> 4.34 mm
- net PD14: track 0.00 -> 4.34 mm
- net PD10: track 0.00 -> 4.34 mm
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Other:
- outline, holes or cut-outs redrawn

Commit message: 100% layout, 90% silkscreen
Parts:
- moved R37 13.2 mm to (176.4, 78.5), turned to 90 degrees
- moved CBY5 10.4 mm to (178.2, 63.8), turned to 180 degrees
- moved U5 0.76 mm to (180.7, 70.3), turned to -90 degrees
Routing:
- net PIXEL+: track 6.55 -> 182.8 mm, vias 0 -> 9
- net PD2_OUT: track 3.92 -> 112.1 mm, vias 0 -> 2
- net PD4_OUT: track 3.92 -> 106.7 mm, vias 0 -> 2
- net PD6_OUT: track 3.92 -> 102.6 mm, vias 0 -> 2
- net PD8_OUT: track 3.92 -> 99.7 mm, vias 0 -> 2
- net PD1_OUT: track 4.28 -> 99.4 mm, vias 0 -> 2
- net PD10_OUT: track 3.92 -> 97.6 mm, vias 0 -> 2
- net PD3_OUT: track 4.28 -> 95.5 mm, vias 0 -> 2
- net PD12_OUT: track 3.92 -> 92.0 mm, vias 0 -> 2
- net PD5_OUT: track 4.28 -> 90.3 mm, vias 0 -> 2
- net PD14_OUT: track 3.92 -> 87.0 mm, vias 0 -> 2
- net PD16_OUT: track 3.92 -> 85.5 mm, vias 0 -> 2
- net PD7_OUT: track 4.28 -> 85.8 mm, vias 0 -> 2
- net PD18_OUT: track 3.92 -> 82.4 mm, vias 0 -> 2
- net PD9_OUT: track 4.28 -> 81.7 mm, vias 0 -> 2
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Other:
- board text added: "+"
- board text added: "-"
- board text added: "MTQ"
- board text added: "PD IN"
- board text added: "PD OUT"
- board text added: "PVDX PAYLOAD BOARD"
- board text added: "PVK"
