File: PVDX-ADCS-PMB.kicad_pcb (KiCad board)
At the start: 4 copper layers, 82.5 x 82.5 mm, 110 parts, among them J1 Conn_02x18_Row_Letter_Last, J2 Conn_01x18, J3 Conn_01x06, J4 Conn_01x02, J5 Conn_01x17, J6 Conn_01x03, J7 Conn_01x09, U1 TLV9001IDCK, U10 DRV8837C, U11 OPA2381AIDGKR, U12 OPA2381AIDGKR, U13 OPA2381AIDGKR, U14 OPA2381AIDGKR, U15 OPA2381AIDGKR, U16 OPA2381AIDGKR, U17 OPA2381AIDGKR, U18 OPA2381AIDGKR, U19 OPA2381AIDGKR, U2 INA226, U3 DRV8837C, U4 DRV8837C, U5 MCP23017x-x-SO, U6 ADG734BRUZ, U7 ADG734BRUZ, U8 ADG734BRUZ, U9 ADG734BRUZ

Commit message: Board complete: 100% silkscreen, repo renamed, NC pins tied; awaiting design review
Parts:
- added G***: LOGO, footprints:snoopy, B.Cu at (160.0, 53.8)
- added G***: LOGO, footprints:hotdog, B.Cu at (150.0, 105.0)
Connections:
- U6 pad 15: unconnected-(U6-NC-Pad15) -> +3V3
- U7 pad 15: unconnected-(U7-NC-Pad15) -> +3V3
- U8 pad 15: unconnected-(U8-NC-Pad15) -> +3V3
- U9 pad 15: unconnected-(U9-NC-Pad15) -> +3V3
Routing:
- net GND: track 107.0 -> 118.7 mm, vias 40 -> 49
- net +3V3: track 82.7 -> 85.3 mm
Other:
- board text added: "1"
- board text added: "1+"
- board text added: "10"
- board text added: "10+"
- board text added: "11"
- board text added: "11+"
- board text added: "12"
- board text added: "12+"
- board text added: "13"
- board text added: "13+"
- board text added: "14"
- board text added: "14+"
- board text added: "15"
- board text added: "15+"
- board text added: "16"
- board text added: "16+"
- board text added: "17"
- board text added: "18"
- board text added: "2"
- board text added: "2+"
- board text added: "3"
- board text added: "3+"
- board text added: "3V3"
- board text added: "4"
- board text added: "4+"
- board text added: "5"
- board text added: "5+"
- board text added: "6"
- board text added: "6+"
- board text added: "7"
- board text added: "7+"
- board text added: "8"
- board text added: "8+"
- board text added: "9"
- board text added: "9+"
- board text added: "DAC"
- board text added: "Designed by Nick Cavallo and Kelly Lin"
- board text added: "GND"
- board text added: "MCU"
- board text added: "Nat"
- board text added: "Nick"
- board text added: "PVDX ADCS/PMB"
- board text added: "PWR"
- board text added: "SCK"
- board text added: "SDA"
- board text added: "X SLP"
- board text added: "X+"
- board text added: "X-"
- board text added: "X1"
- board text added: "X2"
- board text added: "Y SLP"
- board text added: "Y+"
- board text added: "Y-"
- board text added: "Y1"
- board text added: "Y2"
- board text added: "Z SLP"
- board text added: "Z+"
- board text added: "Z-"
- board text added: "Z1"
- board text added: "Z2"
- board text removed: "PVDX PAYLOAD BOARD"

Commit message: silkscreen edits
Parts:
- added G***: LOGO, LOGO, B.Cu at (208.5, 99.6)

Commit message: connect PDGNDs to GND
Parts:
- added NT1: NetTie_2, NetTie:NetTie-2_SMD_Pad0.5mm, F.Cu at (167.5, 114.0)
Connections:
- J1 pad 1: PD1_GND -> PDGND
- J1 pad 11: PD6_GND -> PDGND
- J1 pad 13: PD7_GND -> PDGND
- J1 pad 15: PD8_GND -> PDGND
- J1 pad 17: PD9_GND -> PDGND
- J1 pad 19: PD10_GND -> PDGND
- J1 pad 21: PD11_GND -> PDGND
- J1 pad 23: PD12_GND -> PDGND
- J1 pad 25: PD13_GND -> PDGND
- J1 pad 27: PD14_GND -> PDGND
- J1 pad 29: PD15_GND -> PDGND
- J1 pad 3: PD2_GND -> PDGND
- J1 pad 31: PD16_GND -> PDGND
- J1 pad 33: PD17_GND -> PDGND
- J1 pad 35: PD18_GND -> PDGND
- J1 pad 5: PD3_GND -> PDGND
- J1 pad 7: PD4_GND -> PDGND
- J1 pad 9: PD5_GND -> PDGND
- U11 pad 3: PD1_GND -> PDGND
- U11 pad 5: PD2_GND -> PDGND
- U12 pad 3: PD3_GND -> PDGND
- U12 pad 5: PD4_GND -> PDGND
- U13 pad 3: PD5_GND -> PDGND
- U13 pad 5: PD6_GND -> PDGND
- U14 pad 3: PD7_GND -> PDGND
- U14 pad 5: PD8_GND -> PDGND
- U15 pad 3: PD9_GND -> PDGND
- U15 pad 5: PD10_GND -> PDGND
- U16 pad 3: PD11_GND -> PDGND
- U16 pad 5: PD12_GND -> PDGND
- U17 pad 3: PD13_GND -> PDGND
- U17 pad 5: PD14_GND -> PDGND
- U18 pad 3: PD15_GND -> PDGND
- U18 pad 5: PD16_GND -> PDGND
- U19 pad 3: PD17_GND -> PDGND
- U19 pad 5: PD18_GND -> PDGND
Routing:
- net PDGND: track 0.00 -> 298.3 mm, vias 0 -> 18
- net PD9_GND: track 19.6 -> 0.00 mm, vias 1 -> 0
- net PD7_GND: track 19.5 -> 0.00 mm, vias 1 -> 0
- net PD15_GND: track 19.3 -> 0.00 mm, vias 1 -> 0
- net PD13_GND: track 18.8 -> 0.00 mm, vias 1 -> 0
- net PD1_GND: track 18.5 -> 0.00 mm, vias 1 -> 0
- net PD11_GND: track 18.5 -> 0.00 mm, vias 1 -> 0
- net PD3_GND: track 18.0 -> 0.00 mm, vias 1 -> 0
- net PD17_GND: track 17.8 -> 0.00 mm, vias 1 -> 0
- net PD5_GND: track 17.6 -> 0.00 mm, vias 1 -> 0
- net PD16_GND: track 10.1 -> 0.00 mm, vias 1 -> 0
- net PD18_GND: track 10.1 -> 0.00 mm, vias 1 -> 0
- net PD2_GND: track 9.93 -> 0.00 mm, vias 1 -> 0
- net PD14_GND: track 9.80 -> 0.00 mm, vias 1 -> 0
- net PD4_GND: track 9.59 -> 0.00 mm, vias 1 -> 0
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
Commit message: Prepared for fab: generated gerbers, switched PD C_fb from 22pF to 150pF, generated BOM, updated readme
Parts:
- C45, C46, C47, C48, C49, C50, C51, C52, C53, C54, C55, C56, C57, C58, C59, C60, C61, C62: value 22p -> 150p
Changed lines of the file:
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@@
 		(capping no)
 		(filling no)
+		(zone_defaults)
 		(grid_origin 140 120)
 		(pcbplotparams
@@
 			(plot_on_all_layers_selection 0x00000000_00000000_00000000_00000000)
 			(disableapertmacros no)
-			(usegerberextensions no)
+			(usegerberextensions yes)
 			(usegerberattributes yes)
 			(usegerberadvancedattributes yes)
@@
 			(outputformat 1)
 			(mirror no)
-			(drillshape 1)
+			(drillshape 0)
 			(scaleselection 1)
-			(outputdirectory "")
+			(outputdirectory "manufacturing/rev-1.1_2026-09-04/gerbers/")
 		)
 	)
@@
 			)
 		)
-		(property "Value" "22p"
+		(property "Value" "150p"
 			(at 0 1.43 0)
 			(layer "F.Fab")
@@
 			)
 		)
-		(property "Value" "22p"
+		(property "Value" "150p"
 			(at 0 1.43 0)
 			(layer "F.Fab")
@@
 			)
 		)
-		(property "Value" "22p"
+		(property "Value" "150p"
 			(at 0 1.43 0)
 			(layer "F.Fab")
@@
 			)
 		)
-		(property "Value" "22p"
+		(property "Value" "150p"
 			(at 0 1.43 0)
 			(layer "F.Fab")
@@
 			)
 		)
-		(property "Value" "22p"
+		(property "Value" "150p"
 			(at 0 1.43 0)
 			(layer "F.Fab")
@@
 			)
 		)
-		(property "Value" "22p"
+		(property "Value" "150p"
 			(at 0 1.43 0)
 			(layer "F.Fab")
@@
 			)
 		)
-		(property "Value" "22p"
+		(property "Value" "150p"
 			(at 0 1.43 0)
 			(layer "F.Fab")
@@
 			)
 		)
-		(property "Value" "22p"
+		(property "Value" "150p"
 			(at 0 1.43 0)
 			(layer "F.Fab")
@@
 			)
 		)
-		(property "Value" "22p"
+		(property "Value" "150p"
 			(at 0 1.43 0)
 			(layer "F.Fab")
@@
 			)
 		)
-		(property "Value" "22p"
+		(property "Value" "150p"
 			(at 0 1.43 0)
 			(layer "F.Fab")
@@
 			)
 		)
-		(property "Value" "22p"
+		(property "Value" "150p"
 			(at 0 1.43 0)
 			(layer "F.Fab")
@@
 			)
 		)
-		(property "Value" "22p"
+		(property "Value" "150p"
 			(at 0 1.43 0)
 			(layer "F.Fab")
@@
 			)
 		)
-		(property "Value" "22p"
+		(property "Value" "150p"
 			(at 0 1.43 0)
 			(layer "F.Fab")
@@
 			)
 		)
-		(property "Value" "22p"
+		(property "Value" "150p"
 			(at 0 1.43 0)
 			(layer "F.Fab")
@@
 			)
 		)
-		(property "Value" "22p"
+		(property "Value" "150p"
 			(at 0 1.43 0)
 			(layer "F.Fab")
@@
 			)
 		)
-		(property "Value" "22p"
+		(property "Value" "150p"
 			(at 0 1.43 0)
 			(layer "F.Fab")
@@
 			)
 		)
-		(property "Value" "22p"
+		(property "Value" "150p"
 			(at 0 1.43 0)
 			(layer "F.Fab")
@@
 			)
 		)
-		(property "Value" "22p"
+		(property "Value" "150p"
 			(at 0 1.43 0)
 			(layer "F.Fab")
