File: PVDX-ADCS-PMB.kicad_pcb (KiCad board)
At the start: 4 copper layers, 82.5 x 82.5 mm, 114 parts, among them J1 Conn_02x18_Row_Letter_Last, J2 Conn_01x18, J3 Conn_01x06, J4 Conn_01x02, J5 Conn_01x17, J6 Conn_01x03, J7 Conn_01x09, U1 TLV9001IDCK, U10 DRV8837C, U11 OPA2381AIDGKR, U12 OPA2381AIDGKR, U13 OPA2381AIDGKR, U14 OPA2381AIDGKR, U15 OPA2381AIDGKR, U16 OPA2381AIDGKR, U17 OPA2381AIDGKR, U18 OPA2381AIDGKR, U19 OPA2381AIDGKR, U2 INA226, U3 DRV8837C, U4 DRV8837C, U5 MCP23017x-x-SO, U6 ADG734BRUZ, U7 ADG734BRUZ, U8 ADG734BRUZ, U9 ADG734BRUZ

Commit message: fix BOM, generate .pos, fix component values, re-plot schematics
Parts:
- U1: value TLV9001IDCK -> TLV9001IDCKR
- U10, U3, U4: value DRV8837C -> DRV8837CDSGR
- U2: value INA226 -> INA226AIDGSR
- U5: value MCP23017x-x-SO -> MCP23017-E/SO
