File: PVDX-ADCS-PMB.kicad_sch (KiCad schematic)
At the start: 0 parts

Commit message: fix BOM, generate .pos, fix component values, re-plot schematics
Other:
- title: PVDX ADCS Board -> PVDX ADCS/PMB
Changed lines of the file:
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@@
 	(generator "eeschema")
 	(generator_version "10.0")
-	(paper "A3")
+	(paper "A4")
 	(title_block
-		(title "PVDX ADCS Board")
-		(date "2026-08-06")
+		(title "PVDX ADCS/PMB")
+		(date "2026-09-04")
+		(rev "1.1")
 		(company "Brown Space Engineering")
 	)
