File: schematics/magnetorquers.kicad_sch (KiCad schematic)
At the start: 12 parts, among them U10 DRV8837C, U3 DRV8837C, U4 DRV8837C

Commit message: Board complete: 100% silkscreen, repo renamed, NC pins tied; awaiting design review
Changed lines of the file:
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@@
 	(generator_version "10.0")
 	(paper "A4")
+	(text_box "MTQ Drivers"
+		(exclude_from_sim no)
+		(at 106.68 35.4217 0)
+		(size 13.97 3.9483)
+		(margins 0.9525 0.9525 0.9525 0.9525)
+		(stroke
+			(width 0)
+			(type solid)
+		)
+		(fill
+			(type none)
+		)
+		(effects
+			(font
+				(size 1.27 1.27)
+			)
+		)
+	)
 	(junction
 		(at 114.3 100.33)
@@
 		)
 		(instances
-			(project "PVDX-ADCS-Board"
+			(project "PVDX-ADCS-PMB"
 				(path "/fbb597ca-297a-4338-ae0d-7994cc902267/2dc2922d-9694-40c4-a2c4-76eb44f991c2"
 					(reference "#PWR0113")
@@
 		)
 		(instances
-			(project "PVDX-ADCS-Board"
+			(project "PVDX-ADCS-PMB"
 				(path "/fbb597ca-297a-4338-ae0d-7994cc902267/2dc2922d-9694-40c4-a2c4-76eb44f991c2"
 					(reference "U4")
@@
 		)
 		(instances
-			(project "PVDX-ADCS-Board"
+			(project "PVDX-ADCS-PMB"
 				(path "/fbb597ca-297a-4338-ae0d-7994cc902267/2dc2922d-9694-40c4-a2c4-76eb44f991c2"
 					(reference "C42")
@@
 		)
 		(instances
-			(project "PVDX-ADCS-Board"
+			(project "PVDX-ADCS-PMB"
 				(path "/fbb597ca-297a-4338-ae0d-7994cc902267/2dc2922d-9694-40c4-a2c4-76eb44f991c2"
 					(reference "CB2")
@@
 		)
 		(instances
-			(project "PVDX-ADCS-Board"
+			(project "PVDX-ADCS-PMB"
 				(path "/fbb597ca-297a-4338-ae0d-7994cc902267/2dc2922d-9694-40c4-a2c4-76eb44f991c2"
 					(reference "CB1")
@@
 		)
 		(instances
-			(project "PVDX-ADCS-Board"
+			(project "PVDX-ADCS-PMB"
 				(path "/fbb597ca-297a-4338-ae0d-7994cc902267/2dc2922d-9694-40c4-a2c4-76eb44f991c2"
 					(reference "U10")
@@
 		)
 		(instances
-			(project "PVDX-ADCS-Board"
+			(project "PVDX-ADCS-PMB"
 				(path "/fbb597ca-297a-4338-ae0d-7994cc902267/2dc2922d-9694-40c4-a2c4-76eb44f991c2"
 					(reference "CB3")
@@
 		)
 		(instances
-			(project "PVDX-ADCS-Board"
+			(project "PVDX-ADCS-PMB"
 				(path "/fbb597ca-297a-4338-ae0d-7994cc902267/2dc2922d-9694-40c4-a2c4-76eb44f991c2"
 					(reference "C39")
@@
 		)
 		(instances
-			(project "PVDX-ADCS-Board"
+			(project "PVDX-ADCS-PMB"
 				(path "/fbb597ca-297a-4338-ae0d-7994cc902267/2dc2922d-9694-40c4-a2c4-76eb44f991c2"
 					(reference "#PWR0110")
@@
 		)
 		(instances
-			(project "PVDX-ADCS-Board"
+			(project "PVDX-ADCS-PMB"
 				(path "/fbb597ca-297a-4338-ae0d-7994cc902267/2dc2922d-9694-40c4-a2c4-76eb44f991c2"
 					(reference "#PWR0105")
@@
 		)
 		(instances
-			(project "PVDX-ADCS-Board"
+			(project "PVDX-ADCS-PMB"
 				(path "/fbb597ca-297a-4338-ae0d-7994cc902267/2dc2922d-9694-40c4-a2c4-76eb44f991c2"
 					(reference "U3")
@@
 		)
 		(instances
-			(project "PVDX-ADCS-Board"
+			(project "PVDX-ADCS-PMB"
 				(path "/fbb597ca-297a-4338-ae0d-7994cc902267/2dc2922d-9694-40c4-a2c4-76eb44f991c2"
 					(reference "#PWR093")
@@
 		)
 		(instances
-			(project "PVDX-ADCS-Board"
+			(project "PVDX-ADCS-PMB"
 				(path "/fbb597ca-297a-4338-ae0d-7994cc902267/2dc2922d-9694-40c4-a2c4-76eb44f991c2"
 					(reference "#PWR086")
@@
 		)
 		(instances
-			(project "PVDX-ADCS-Board"
+			(project "PVDX-ADCS-PMB"
 				(path "/fbb597ca-297a-4338-ae0d-7994cc902267/2dc2922d-9694-40c4-a2c4-76eb44f991c2"
 					(reference "C40")
@@
 		)
 		(instances
-			(project "PVDX-ADCS-Board"
+			(project "PVDX-ADCS-PMB"
 				(path "/fbb597ca-297a-4338-ae0d-7994cc902267/2dc2922d-9694-40c4-a2c4-76eb44f991c2"
 					(reference "#PWR0109")
@@
 		)
 		(instances
-			(project "PVDX-ADCS-Board"
+			(project "PVDX-ADCS-PMB"
 				(path "/fbb597ca-297a-4338-ae0d-7994cc902267/2dc2922d-9694-40c4-a2c4-76eb44f991c2"
 					(reference "#PWR099")
@@
 		)
 		(instances
-			(project "PVDX-ADCS-Board"
+			(project "PVDX-ADCS-PMB"
 				(path "/fbb597ca-297a-4338-ae0d-7994cc902267/2dc2922d-9694-40c4-a2c4-76eb44f991c2"
 					(reference "#PWR084")
@@
 		)
 		(instances
-			(project "PVDX-ADCS-Board"
+			(project "PVDX-ADCS-PMB"
 				(path "/fbb597ca-297a-4338-ae0d-7994cc902267/2dc2922d-9694-40c4-a2c4-76eb44f991c2"
 					(reference "#PWR0114")
@@
 		)
 		(instances
-			(project "PVDX-ADCS-Board"
+			(project "PVDX-ADCS-PMB"
 				(path "/fbb597ca-297a-4338-ae0d-7994cc902267/2dc2922d-9694-40c4-a2c4-76eb44f991c2"
 					(reference "#PWR085")
@@
 		)
 		(instances
-			(project "PVDX-ADCS-Board"
+			(project "PVDX-ADCS-PMB"
 				(path "/fbb597ca-297a-4338-ae0d-7994cc902267/2dc2922d-9694-40c4-a2c4-76eb44f991c2"
 					(reference "#PWR087")
@@
 		)
 		(instances
-			(project "PVDX-ADCS-Board"
+			(project "PVDX-ADCS-PMB"
 				(path "/fbb597ca-297a-4338-ae0d-7994cc902267/2dc2922d-9694-40c4-a2c4-76eb44f991c2"
 					(reference "C37")
@@
 		)
 		(instances
-			(project "PVDX-ADCS-Board"
+			(project "PVDX-ADCS-PMB"
 				(path "/fbb597ca-297a-4338-ae0d-7994cc902267/2dc2922d-9694-40c4-a2c4-76eb44f991c2"
 					(reference "C41")
@@
 		)
 		(instances
-			(project "PVDX-ADCS-Board"
+			(project "PVDX-ADCS-PMB"
 				(path "/fbb597ca-297a-4338-ae0d-7994cc902267/2dc2922d-9694-40c4-a2c4-76eb44f991c2"
 					(reference "C38")
@@
 		)
 		(instances
-			(project "PVDX-ADCS-Board"
+			(project "PVDX-ADCS-PMB"
 				(path "/fbb597ca-297a-4338-ae0d-7994cc902267/2dc2922d-9694-40c4-a2c4-76eb44f991c2"
 					(reference "#PWR045")

Commit message: fix BOM, generate .pos, fix component values, re-plot schematics
Parts:
- U10, U3, U4: value DRV8837C -> DRV8837CDSGR; Manufacturer_Name (none) -> Texas Instruments; Manufacturer_Part_Number (none) -> DRV8837CDSGR
Other:
- company: (none) -> Brown Space Engineering
- title: (none) -> PVDX ADCS/PMB
Changed lines of the file:
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@@
 	(generator_version "10.0")
 	(paper "A4")
+	(title_block
+		(title "PVDX ADCS/PMB")
+		(date "2026-09-04")
+		(rev "1.1")
+		(company "Brown Space Engineering")
+	)
 	(text_box "MTQ Drivers"
 		(exclude_from_sim no)
@@
 			)
 		)
-		(property "Value" "DRV8837C"
+		(property "Value" "DRV8837CDSGR"
 			(at 116.4433 128.27 0)
 			(show_name no)
@@
 		)
 		(property "Description" "H-Bridge driver, 1A, Low Voltage, PWM input, WSON-8"
+			(at 114.3 113.03 0)
+			(hide yes)
+			(show_name no)
+			(do_not_autoplace no)
+			(effects
+				(font
+					(size 1.27 1.27)
+				)
+			)
+		)
+		(property "Manufacturer_Name" "Texas Instruments"
+			(at 114.3 113.03 0)
+			(hide yes)
+			(show_name no)
+			(do_not_autoplace no)
+			(effects
+				(font
+					(size 1.27 1.27)
+				)
+			)
+		)
+		(property "Manufacturer_Part_Number" "DRV8837CDSGR"
 			(at 114.3 113.03 0)
 			(hide yes)
@@
 			)
 		)
-		(property "Value" "DRV8837C"
+		(property "Value" "DRV8837CDSGR"
 			(at 116.4433 175.26 0)
 			(show_name no)
@@
 		)
 		(property "Description" "H-Bridge driver, 1A, Low Voltage, PWM input, WSON-8"
+			(at 114.3 160.02 0)
+			(hide yes)
+			(show_name no)
+			(do_not_autoplace no)
+			(effects
+				(font
+					(size 1.27 1.27)
+				)
+			)
+		)
+		(property "Manufacturer_Name" "Texas Instruments"
+			(at 114.3 160.02 0)
+			(hide yes)
+			(show_name no)
+			(do_not_autoplace no)
+			(effects
+				(font
+					(size 1.27 1.27)
+				)
+			)
+		)
+		(property "Manufacturer_Part_Number" "DRV8837CDSGR"
 			(at 114.3 160.02 0)
 			(hide yes)
@@
 			)
 		)
-		(property "Value" "DRV8837C"
+		(property "Value" "DRV8837CDSGR"
 			(at 116.4433 82.55 0)
 			(show_name no)
@@
 			(at 114.3 67.31 0)
 			(hide yes)
+			(show_name no)
+			(do_not_autoplace no)
+			(effects
+				(font
+					(size 1.27 1.27)
+				)
+			)
+		)
+		(property "Manufacturer_Name" "Texas Instruments"
+			(at 114.3 67.31 0)
+			(hide yes)
+			(show_name no)
+			(do_not_autoplace no)
+			(effects
+				(font
+					(size 1.27 1.27)
+				)
+			)
+		)
+		(property "Manufacturer_Part_Number" "DRV8837CDSGR"
+			(at 114.3 67.31 0)
+			(hide yes)
