File: schematics/perovskites.kicad_sch (KiCad schematic)
At the start: 33 parts, among them U1 TLV9001IDCK, U2 INA226, U5 MCP23017x-x-SO, U6 ADG734BRUZ, U7 ADG734BRUZ, U8 ADG734BRUZ, U9 ADG734BRUZ

Commit message: Board complete: 100% silkscreen, repo renamed, NC pins tied; awaiting design review
Connections:
- net +3V3: now also U6.15 (NC), U7.15 (NC), U8.15 (NC), U9.15 (NC)
- no-connect marks 7 -> 3
Other:
- moved on the sheet: CBY2, CBY8, R10, R11, R12, R13, R14, R15, R18, R3, R6, R7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

Commit message: fix BOM, generate .pos, fix component values, re-plot schematics
Parts:
- R1: Manufacturer_Name (none) -> Bourns Inc.; Manufacturer_Part_Number (none) -> CRT0603-BY-2102ELF
- R10, R11, R12, R13, R14, R15, R16, R17, R18, R3, R4, R5, R6, R7, R8, R9: Manufacturer_Name (none) -> Panasonic Industry; Manufacturer_Part_Number (none) -> ERJ-3EKF1000V
- R2: Manufacturer_Name (none) -> Bourns Inc.; Manufacturer_Part_Number (none) -> CRT0603-BY-1202ELF
- RSH1: Manufacturer_Name (none) -> Bourns Inc.; Manufacturer_Part_Number (none) -> CRT0603-BY-10R0ELF
- U1: value TLV9001IDCK -> TLV9001IDCKR; Manufacturer_Name (none) -> Texas Instruments; Manufacturer_Part_Number (none) -> TLV9001IDCKR
- U2: value INA226 -> INA226AIDGSR; Manufacturer_Name (none) -> Texas Instruments; Manufacturer_Part_Number (none) -> INA226AIDGSR
- U5: value MCP23017x-x-SO -> MCP23017-E/SO; Manufacturer_Name (none) -> Microchip Technology; Manufacturer_Part_Number (none) -> MCP23017-E/SO
- U6, U7, U8, U9: Manufacturer_Name (none) -> Analog Devices Inc.; Manufacturer_Part_Number (none) -> ADG734BRUZ
Other:
- company: (none) -> Brown Space Engineering
- title: (none) -> PVDX ADCS/PMB
